Commit message: modify mesh file save location

File: MFFRUnity/Assets/TemporaryRobotDescription/temporary_robot.urdf (robot description, URDF)
Before this commit: robot test_robot, 8 links, 7 joints
Links:
- removed link base_link
- removed link link_1
- removed link link_2
- removed link link_3
- removed link link_4
- removed link link_5
- removed link link_6
- added link base_rail_link, mass 1.0; collision mesh filename=mesh/base_rail_link.stl; visual mesh filename=mesh/base_rail_link.stl
- added link link_01, mass 1.0; collision mesh filename=mesh/link_01.stl; visual mesh filename=mesh/link_01.stl
- added link link_02, mass 1.0; collision mesh filename=mesh/link_02.stl; visual mesh filename=mesh/link_02.stl
- added link link_03, mass 1.0; collision mesh filename=mesh/link_03.stl; visual mesh filename=mesh/link_03.stl
- added link link_04, mass 1.0; collision mesh filename=mesh/link_04.stl; visual mesh filename=mesh/link_04.stl
- added link link_05, mass 1.0; collision mesh filename=mesh/link_05.stl; visual mesh filename=mesh/link_05.stl
- added link link_06, mass 1.0; collision mesh filename=mesh/link_06.stl; visual mesh filename=mesh/link_06.stl
- added link link_07, mass 1.0; collision mesh filename=mesh/link_07.stl; visual mesh filename=mesh/link_07.stl
- added link link_08, mass 1.0; collision mesh filename=mesh/link_08.stl; visual mesh filename=mesh/link_08.stl
- added link link_09, mass 1.0; collision mesh filename=mesh/link_09.stl; visual mesh filename=mesh/link_09.stl
- added link link_10, mass 1.0; collision mesh filename=mesh/link_10.stl; visual mesh filename=mesh/link_10.stl
Joints:
- removed joint joint_0
- removed joint joint_1
- removed joint joint_2
- removed joint joint_3
- removed joint joint_4
- removed joint joint_5
- added joint joint_01: type prismatic, parent base_rail_link, child link_01, origin xyz=0.0 0.0 0.375 rpy=0.0 0.0 0.0, axis 0 1 0, limit lower=-3.141592653589793 upper=3.141592653589793 effort=100.0 velocity=1.0
- added joint joint_02: type revolute, parent link_01, child link_02, origin xyz=0.0 1.0 0.0 rpy=0 0 0, axis 0 0 1, limit lower=-3.141592653589793 upper=3.141592653589793 effort=100.0 velocity=1.0
- added joint joint_03: type revolute, parent link_02, child link_03, origin xyz=0.0 1.41 0.0 rpy=0 0 0, axis 0 0 1, limit lower=-3.141592653589793 upper=3.141592653589793 effort=100.0 velocity=1.0
- added joint joint_04: type revolute, parent link_03, child link_04, origin xyz=0.0 1.13 0.0 rpy=0 0 0, axis 0 1 0, limit lower=-3.141592653589793 upper=3.141592653589793 effort=100.0 velocity=1.0
- added joint joint_05: type revolute, parent link_04, child link_05, origin xyz=0.0 0.565257 0.356751 rpy=0.0 0.0 3.141592653589793, axis 1 0 0, limit lower=-3.141592653589793 upper=3.141592653589793 effort=100.0 velocity=1.0
- added joint joint_06: type revolute, parent link_05, child link_06, origin xyz=0.0 0.86 0.39 rpy=0 0 0, axis 0 1 0, limit lower=-3.141592653589793 upper=3.141592653589793 effort=100.0 velocity=1.0
- added joint joint_07: type revolute, parent link_06, child link_07, origin xyz=0.0 1.175 0.0 rpy=0 0 0, axis 0 0 1, limit lower=-3.141592653589793 upper=3.141592653589793 effort=100.0 velocity=1.0
- added joint joint_08: type revolute, parent link_07, child link_08, origin xyz=0.0 0.62 0.0 rpy=0 0 0, axis 0 1 0, limit lower=-3.141592653589793 upper=3.141592653589793 effort=100.0 velocity=1.0
- added joint joint_09: type revolute, parent link_08, child link_09, origin xyz=0.0 0.68 0.2 rpy=-1.5707963267948966 0.0 0.0, axis 1 0 0, limit lower=-3.141592653589793 upper=3.141592653589793 effort=100.0 velocity=1.0
- added joint joint_10: type revolute, parent link_09, child link_10, origin xyz=0.0 0.0 0.65 rpy=0.0 0.0 0.0, axis 0 0 1, limit lower=-3.141592653589793 upper=3.141592653589793 effort=100.0 velocity=1.0
- joint world_joint: child base_link -> base_rail_link

Commit message: add various functions and scripts

File: MFFRUnity/Assets/TemporaryRobotDescription/temporary_robot.urdf (robot description, URDF)
Before this commit: robot test_robot, 12 links, 11 joints
Links:
- link base_rail_link: geometry collision mesh filename=collision/base_rail_link_col.stl; visual mesh filename=mesh/base_rail_link.stl
- link link_01: geometry collision mesh filename=collision/link_01_col.stl; visual mesh filename=mesh/link_01.stl
- link link_02: geometry collision mesh filename=collision/link_02_col.stl; visual mesh filename=mesh/link_02.stl
- link link_03: geometry collision mesh filename=collision/link_03_col.stl; visual mesh filename=mesh/link_03.stl
- link link_04: geometry collision mesh filename=collision/link_04_col.stl; visual mesh filename=mesh/link_04.stl
- link link_05: geometry collision mesh filename=collision/link_05_col.stl; visual mesh filename=mesh/link_05.stl
- link link_06: geometry collision mesh filename=collision/link_06_col.stl; visual mesh filename=mesh/link_06.stl
- link link_07: geometry collision mesh filename=collision/link_07_col.stl; visual mesh filename=mesh/link_07.stl
- link link_08: geometry collision mesh filename=collision/link_08_col.stl; visual mesh filename=mesh/link_08.stl
- link link_09: geometry collision mesh filename=collision/link_09_col.stl; visual mesh filename=mesh/link_09.stl
- link link_10: geometry collision mesh filename=collision/link_10_col.stl; visual mesh filename=mesh/link_10.stl
